Commit message: gazebo completed

File: panda_description/urdf/backup/segway_e1.xacro (robot description, xacro)
@@ -1,8 +1,9 @@
 <?xml version="1.0"?>
 <robot name="segway" xmlns:xacro="http://www.ros.org/wiki/xacro">
-    <xacro:include filename="/home/plus/Work/segway_ws/src/segway_e1_description/urdf/segway_e1_body.xacro" />
-    <xacro:include filename="/home/plus/Work/segway_ws/src/segway_e1_description/urdf/segway_transmission.xacro" />
+    <xacro:include filename="$(find panda_description)/urdf/segway_e1_body.xacro" />
+    <xacro:include filename="$(find panda_description)/urdf/segway_transmission.xacro" />
     <xacro:wheel_transmission LR="right" FR="rear"/>
     <xacro:wheel_transmission LR="left" FR="rear"/>
+    <xacro:steering_transmission />
     <!-- <wheel_transmission LR="right" FR="front"/>
     <wheel_transmission LR="left" FR="front"/> -->

File: panda_description/urdf/backup/segway_e1_body.xacro (robot description, xacro)
@@ -33,19 +33,19 @@
       <geometry>
         <mesh
-          filename="package://segway_e1_description/meshes/Chassis body.STL" />
-      </geometry>
-      <material
-        name="">
-        <color
-          rgba="0.79216 0.81961 0.93333 1" />
-      </material>
-    </visual>
-    <collision>
-      <origin
-        xyz="0 0 0"
-        rpy="0 0 0" />
-      <geometry>
-        <mesh
-          filename="package://segway_e1_description/meshes/Chassis body.STL" />
+          filename="package://panda_description/meshes/Chassis body.STL" />
+      </geometry>
+      <material
+        name="">
+        <color
+          rgba="0.79216 0.81961 0.93333 1" />
+      </material>
+    </visual>
+    <collision>
+      <origin
+        xyz="0 0 0"
+        rpy="0 0 0" />
+      <geometry>
+        <mesh
+          filename="package://panda_description/meshes/Chassis body.STL" />
       </geometry>
     </collision>
@@ -78,19 +78,19 @@
       <geometry>
         <mesh
-          filename="package://segway_e1_description/meshes/Wheel.STL" />
-      </geometry>
-      <material
-        name="">
-        <color
-          rgba="0.79216 0.81961 0.93333 1" />
-      </material>
-    </visual>
-    <collision>
-      <origin
-        xyz="0 0 0"
-        rpy="0 0 0" />
-      <geometry>
-        <mesh
-          filename="package://segway_e1_description/meshes/Wheel.STL" />
+          filename="package://panda_description/meshes/Wheel.STL" />
+      </geometry>
+      <material
+        name="">
+        <color
+          rgba="0.79216 0.81961 0.93333 1" />
+      </material>
+    </visual>
+    <collision>
+      <origin
+        xyz="0 0 0"
+        rpy="0 0 0" />
+      <geometry>
+        <mesh
+          filename="package://panda_description/meshes/Wheel.STL" />
       </geometry>
     </collision>
@@ -131,19 +131,19 @@
       <geometry>
         <mesh
-          filename="package://segway_e1_description/meshes/Wheel.STL" />
-      </geometry>
-      <material
-        name="">
-        <color
-          rgba="0.79216 0.81961 0.93333 1" />
-      </material>
-    </visual>
-    <collision>
-      <origin
-        xyz="0 0 0"
-        rpy="0 0 0" />
-      <geometry>
-        <mesh
-          filename="package://segway_e1_description/meshes/Wheel.STL" />
+          filename="package://panda_description/meshes/Wheel.STL" />
+      </geometry>
+      <material
+        name="">
+        <color
+          rgba="0.79216 0.81961 0.93333 1" />
+      </material>
+    </visual>
+    <collision>
+      <origin
+        xyz="0 0 0"
+        rpy="0 0 0" />
+      <geometry>
+        <mesh
+          filename="package://panda_description/meshes/Wheel.STL" />
       </geometry>
     </collision>
@@ -184,19 +184,19 @@
       <geometry>
         <mesh
-          filename="package://segway_e1_description/meshes/Chassis front beam.STL" />
-      </geometry>
-      <material
-        name="">
-        <color
-          rgba="0.79216 0.81961 0.93333 1" />
-      </material>
-    </visual>
-    <collision>
-      <origin
-        xyz="0 0 0"
-        rpy="0 0 0" />
-      <geometry>
-        <mesh
-          filename="package://segway_e1_description/meshes/Chassis front beam.STL" />
+          filename="package://panda_description/meshes/Chassis front beam.STL" />
+      </geometry>
+      <material
+        name="">
+        <color
+          rgba="0.79216 0.81961 0.93333 1" />
+      </material>
+    </visual>
+    <collision>
+      <origin
+        xyz="0 0 0"
+        rpy="0 0 0" />
+      <geometry>
+        <mesh
+          filename="package://panda_description/meshes/Chassis front beam.STL" />
       </geometry>
     </collision>
@@ -242,19 +242,19 @@
       <geometry>
         <mesh
-          filename="package://segway_e1_description/meshes/Wheel.STL" />
-      </geometry>
-      <material
-        name="">
-        <color
-          rgba="0.79216 0.81961 0.93333 1" />
-      </material>
-    </visual>
-    <collision>
-      <origin
-        xyz="0 0 0"
-        rpy="0 0 0" />
-      <geometry>
-        <mesh
-          filename="package://segway_e1_description/meshes/Wheel.STL" />
+          filename="package://panda_description/meshes/Wheel.STL" />
+      </geometry>
+      <material
+        name="">
+        <color
+          rgba="0.79216 0.81961 0.93333 1" />
+      </material>
+    </visual>
+    <collision>
+      <origin
+        xyz="0 0 0"
+        rpy="0 0 0" />
+      <geometry>
+        <mesh
+          filename="package://panda_description/meshes/Wheel.STL" />
       </geometry>
     </collision>
@@ -295,19 +295,19 @@
       <geometry>
         <mesh
-          filename="package://segway_e1_description/meshes/Wheel.STL" />
-      </geometry>
-      <material
-        name="">
-        <color
-          rgba="0.79216 0.81961 0.93333 1" />
-      </material>
-    </visual>
-    <collision>
-      <origin
-        xyz="0 0 0"
-        rpy="0 0 0" />
-      <geometry>
-        <mesh
-          filename="package://segway_e1_description/meshes/Wheel.STL" />
+          filename="package://panda_description/meshes/Wheel.STL" />
+      </geometry>
+      <material
+        name="">
+        <color
+          rgba="0.79216 0.81961 0.93333 1" />
+      </material>
+    </visual>
+    <collision>
+      <origin
+        xyz="0 0 0"
+        rpy="0 0 0" />
+      <geometry>
+        <mesh
+          filename="package://panda_description/meshes/Wheel.STL" />
       </geometry>
     </collision>

File: panda_description/urdf/backup/segway_transmission.xacro (robot description, xacro)
@@ -29,16 +29,16 @@
     </transmission>
     </xacro:macro>
-    <!-- <xacro:macro name="steering_transmission" params="LR">
-    <transmission name="${LR}_steering_trans">
+    <xacro:macro name="steering_transmission">
+    <transmission name="steering_trans">
       <type>transmission_interface/SimpleTransmission</type>
-      <joint name="${LR}_steering_joint">
-        <hardwareInterface>PositionJointInterface</hardwareInterface>
+      <joint name="Chassis_front_joint">
+        <hardwareInterface>hardware_interface/EffortJointInterface</hardwareInterface>
       </joint>
-      <actuator name="${LR}_steering_act">
-        <hardwareInterface>PositionJointInterface</hardwareInterface>
+      <actuator name="Chassis_front_joint">
+        <hardwareInterface>hardware_interface/EffortJointInterface</hardwareInterface>
         <mechanicalReduction>1</mechanicalReduction>
       </actuator>
     </transmission>
-    </xacro:macro> -->
+    </xacro:macro>
 <!-- Defining the control plugin used in this robot -->
   <gazebo>

File: panda_description/urdf/panda_body.xacro (robot description, xacro)
@@ -1,8 +1,12 @@
-<?xml version="1.0" encoding="utf-8"?>
-<!-- This URDF was automatically created by SolidWorks to URDF Exporter! Originally created by Stephen Brawner (brawner@gmail.com)
-     Commit Version: 1.5.1-0-g916b5db  Build Version: 1.5.7152.31018
-     For more information, please see http://wiki.ros.org/sw_urdf_exporter -->
-<robot
-  name="segway_e1_description">
+<?xml version="1.0"?>
+<robot name="segway" xmlns:xacro="http://www.ros.org/wiki/xacro">
+  <xacro:macro name="Box_inertial_matrix" params="m l w h">
+       <inertial>
+               <mass value="${m}" />
+               <inertia ixx="${m*(h*h + l*l)/12}" ixy = "0" ixz = "0"
+                   iyy="${m*(w*w + l*l)/12}" iyz= "0"
+                   izz="${m*(w*w + h*h)/12}" />
+       </inertial>
+   </xacro:macro>
   <link name="base_link"/>
   <link
@@ -14,4 +18,5 @@
       <mass
         value="1.5192" />
+      <!-- <xacro:Box_inertial_matrix m="1.5192" l="0.6" w="0.1" h="0.1" /> -->
       <inertia
         ixx="0.048829"
@@ -21,26 +26,26 @@
         iyz="-0.002399"
         izz="0.052057" />
-    </inertial>
-    <visual>
-      <origin
-        xyz="0 0 0"
-        rpy="0 0 0" />
-      <geometry>
-        <mesh
-          filename="package://segway_e1_description/meshes/Chassis body.STL" />
-      </geometry>
-      <material
-        name="">
-        <color
-          rgba="0.79216 0.81961 0.93333 1" />
-      </material>
-    </visual>
-    <collision>
-      <origin
-        xyz="0 0 0"
-        rpy="0 0 0" />
-      <geometry>
-        <mesh
-          filename="package://segway_e1_description/meshes/Chassis body.STL" />
+      </inertial>
+    <visual>
+      <origin
+        xyz="0 0 0"
+        rpy="0 0 0" />
+      <geometry>
+        <mesh
+          filename="package://panda_description/meshes/Chassis body.STL" />
+      </geometry>
+      <material
+        name="">
+        <color
+          rgba="0.79216 0.81961 0.93333 1" />
+      </material>
+    </visual>
+    <collision>
+      <origin
+        xyz="0 0 0"
+        rpy="0 0 0" />
+      <geometry>
+        <mesh
+          filename="package://panda_description/meshes/Chassis body.STL" />
       </geometry>
     </collision>
@@ -73,24 +78,24 @@
       <geometry>
         <mesh
-          filename="package://segway_e1_description/meshes/Wheel.STL" />
-      </geometry>
-      <material
-        name="">
-        <color
-          rgba="0.79216 0.81961 0.93333 1" />
-      </material>
-    </visual>
-    <collision>
-      <origin
-        xyz="0 0 0"
-        rpy="0 0 0" />
-      <geometry>
-        <mesh
-          filename="package://segway_e1_description/meshes/Wheel.STL" />
-      </geometry>
-    </collision>
-  </link>
-  <joint
-    name="Left_rear"
+          filename="package://panda_description/meshes/Wheel.STL" />
+      </geometry>
+      <material
+        name="">
+        <color
+          rgba="0.79216 0.81961 0.93333 1" />
+      </material>
+    </visual>
+    <collision>
+      <origin
+        xyz="0 0 0"
+        rpy="0 0 0" />
+      <geometry>
+        <mesh
+          filename="package://panda_description/meshes/Wheel.STL" />
+      </geometry>
+    </collision>
+  </link>
+  <joint
+    name="left_rear_wheel_joint"
     type="continuous">
     <origin
@@ -126,24 +131,24 @@
       <geometry>
         <mesh
-          filename="package://segway_e1_description/meshes/Wheel.STL" />
-      </geometry>
-      <material
-        name="">
-        <color
-          rgba="0.79216 0.81961 0.93333 1" />
-      </material>
-    </visual>
-    <collision>
-      <origin
-        xyz="0 0 0"
-        rpy="0 0 0" />
-      <geometry>
-        <mesh
-          filename="package://segway_e1_description/meshes/Wheel.STL" />
-      </geometry>
-    </collision>
-  </link>
-  <joint
-    name="Right_rear"
+          filename="package://panda_description/meshes/Wheel.STL" />
+      </geometry>
+      <material
+        name="">
+        <color
+          rgba="0.79216 0.81961 0.93333 1" />
+      </material>
+    </visual>
+    <collision>
+      <origin
+        xyz="0 0 0"
+        rpy="0 0 0" />
+      <geometry>
+        <mesh
+          filename="package://panda_description/meshes/Wheel.STL" />
+      </geometry>
+    </collision>
+  </link>
+  <joint
+    name="right_rear_wheel_joint"
     type="continuous">
     <origin
@@ -179,24 +184,24 @@
       <geometry>
         <mesh
-          filename="package://segway_e1_description/meshes/Chassis front beam.STL" />
-      </geometry>
-      <material
-        name="">
-        <color
-          rgba="0.79216 0.81961 0.93333 1" />
-      </material>
-    </visual>
-    <collision>
-      <origin
-        xyz="0 0 0"
-        rpy="0 0 0" />
-      <geometry>
-        <mesh
-          filename="package://segway_e1_description/meshes/Chassis front beam.STL" />
-      </geometry>
-    </collision>
-  </link>
-  <joint
-    name="Chassis_front_joint"
+          filename="package://panda_description/meshes/Chassis front beam.STL" />
+      </geometry>
+      <material
+        name="">
+        <color
+          rgba="0.79216 0.81961 0.93333 1" />
+      </material>
+    </visual>
+    <collision>
+      <origin
+        xyz="0 0 0"
+        rpy="0 0 0" />
+      <geometry>
+        <mesh
+          filename="package://panda_description/meshes/Chassis front beam.STL" />
+      </geometry>
+    </collision>
+  </link>
+  <joint
+    name="chassis_front_steer_joint"
     type="revolute">
     <origin
@@ -237,24 +242,24 @@
       <geometry>
         <mesh
-          filename="package://segway_e1_description/meshes/Wheel.STL" />
-      </geometry>
-      <material
-        name="">
-        <color
-          rgba="0.79216 0.81961 0.93333 1" />
-      </material>
-    </visual>
-    <collision>
-      <origin
-        xyz="0 0 0"
-        rpy="0 0 0" />
-      <geometry>
-        <mesh
-          filename="package://segway_e1_description/meshes/Wheel.STL" />
-      </geometry>
-    </collision>
-  </link>
-  <joint
-    name="Left_front"
+          filename="package://panda_description/meshes/Wheel.STL" />
+      </geometry>
+      <material
+        name="">
+        <color
+          rgba="0.79216 0.81961 0.93333 1" />
+      </material>
+    </visual>
+    <collision>
+      <origin
+        xyz="0 0 0"
+        rpy="0 0 0" />
+      <geometry>
+        <mesh
+          filename="package://panda_description/meshes/Wheel.STL" />
+      </geometry>
+    </collision>
+  </link>
+  <joint
+    name="left_front_wheel_joint"
     type="continuous">
     <origin
@@ -290,24 +295,24 @@
       <geometry>
         <mesh
-          filename="package://segway_e1_description/meshes/Wheel.STL" />
-      </geometry>
-      <material
-        name="">
-        <color
-          rgba="0.79216 0.81961 0.93333 1" />
-      </material>
-    </visual>
-    <collision>
-      <origin
-        xyz="0 0 0"
-        rpy="0 0 0" />
-      <geometry>
-        <mesh
-          filename="package://segway_e1_description/meshes/Wheel.STL" />
-      </geometry>
-    </collision>
-  </link>
-  <joint
-    name="Right_front"
+          filename="package://panda_description/meshes/Wheel.STL" />
+      </geometry>
+      <material
+        name="">
+        <color
+          rgba="0.79216 0.81961 0.93333 1" />
+      </material>
+    </visual>
+    <collision>
+      <origin
+        xyz="0 0 0"
+        rpy="0 0 0" />
+      <geometry>
+        <mesh
+          filename="package://panda_description/meshes/Wheel.STL" />
+      </geometry>
+    </collision>
+  </link>
+  <joint
+    name="right_front_wheel_joint"
     type="continuous">
     <origin
